Commit message: Updated

File: niryo_one_description/urdf/niryo_one_gripper.urdf.xacro (robot description, xacro)
@@ -89,4 +89,5 @@
                effort="1"
                velocity="5"/>
+        <mimic joint="${prefix}_gripper_joint" multiplier="1" offset="0" />
     </joint>
     <!-- Mors 2 -->
@@ -133,5 +134,17 @@
                effort="1"
                velocity="5"/>
+        <mimic joint="${prefix}_joint_base_to_mors_1" multiplier="1" offset="0" />
     </joint>
+    <ros2_control name="${prefix}_gripper" type="actuator">
+      <hardware>
+        <plugin>niryo_one_driver/NiryoOneActuatorInterface</plugin>
+      </hardware>
+      <joint name="${prefix}_joint_base_to_mors_1">
+        <command_interface name="position"/>
+        <state_interface name="position"/>
+        <state_interface name="velocity"/>
+        <state_interface name="effort"/>
+      </joint>
+    </ros2_control>
     <xacro:macro name="SimpleTransmissionEffort" params="joint n">
     <transmission name="${prefix}_transmission_${n}">

File: niryo_one_moveit_config/srdf/niryo_two.srdf.xacro (robot description, xacro)
@@ -18,6 +18,6 @@
         <joint name="a_bot_joint_5"/>
         <joint name="a_bot_joint_6"/>
-        <joint name="a_bot_hand_tool_joint"/>
-        <chain base_link="a_bot_base_link" tip_link="a_bot_tool_link"/>
+        <link name="a_bot_hand_link"/>
+        <link name="a_bot_tool_link"/>
     </group>
     <group name="b_bot">
@@ -29,6 +29,6 @@
         <joint name="b_bot_joint_5"/>
         <joint name="b_bot_joint_6"/>
-        <joint name="b_bot_hand_tool_joint"/>
-        <chain base_link="b_bot_base_link" tip_link="b_bot_tool_link"/>
+        <link name="b_bot_hand_link"/>
+        <link name="b_bot_tool_link"/>
     </group>
     <group name="niryo_two">
@@ -40,13 +40,10 @@
         <joint name="a_bot_joint_to_gripper"/>
         <joint name="a_bot_joint_base_to_mors_1"/>
-        <joint name="a_bot_joint_base_to_mors_2"/>
     </group>
     <group_state name="close" group="a_bot_tool">
         <joint name="a_bot_joint_base_to_mors_1" value="-0.01"/>
-        <joint name="a_bot_joint_base_to_mors_2" value="-0.01"/>
     </group_state>
     <group_state name="open" group="a_bot_tool">
         <joint name="a_bot_joint_base_to_mors_1" value="0.007"/>
-        <joint name="a_bot_joint_base_to_mors_2" value="0.007"/>
     </group_state>
     <group name="b_bot_tool">
@@ -54,13 +51,10 @@
         <joint name="b_bot_joint_to_gripper"/>
         <joint name="b_bot_joint_base_to_mors_1"/>
-        <joint name="b_bot_joint_base_to_mors_2"/>
     </group>
     <group_state name="close" group="b_bot_tool">
-        <joint name="a_bot_joint_base_to_mors_1" value="-0.01"/>
-        <joint name="a_bot_joint_base_to_mors_2" value="-0.01"/>
+        <joint name="b_bot_joint_base_to_mors_1" value="-0.01"/>
     </group_state>
     <group_state name="open" group="b_bot_tool">
         <joint name="b_bot_joint_base_to_mors_1" value="0.007"/>
-        <joint name="b_bot_joint_base_to_mors_2" value="0.007"/>
     </group_state>
     <!--VIRTUAL JOINT Purpose this element defines a virtual joint between a robot link and an external frame of reference (considered fixed with respect to the robot)-->
