Commit message: Final update for examples

File: niryo_one_description/urdf/bot.xacro (robot description, xacro)
@@ -244,38 +244,5 @@
         <origin xyz="0 0 ${distance_hand_tool}" rpy="${-PI/2} ${-PI/2} 0" />
 	</joint>
-    <ros2_control name="${name}" type="system">
-      <hardware>
-        <plugin>niryo_one_driver/NiryoOneHardwareInterface</plugin>
-      </hardware>
-      <joint name="${prefix}_joint_1">
-        <command_interface name="position"/>
-        <state_interface name="position"/>
-        <state_interface name="velocity"/>
-      </joint>
-      <joint name="${prefix}_joint_2">
-        <command_interface name="position"/>
-        <state_interface name="position"/>
-        <state_interface name="velocity"/>
-      </joint>
-        <joint name="${prefix}_joint_3">
-        <command_interface name="position"/>
-        <state_interface name="position"/>
-        <state_interface name="velocity"/>
-      </joint>
-        <joint name="${prefix}_joint_4">
-        <command_interface name="position"/>
-        <state_interface name="position"/>
-        <state_interface name="velocity"/>
-      </joint>
-        <joint name="${prefix}_joint_5">
-        <command_interface name="position"/>
-        <state_interface name="position"/>
-        <state_interface name="velocity"/>
-      </joint>
-        <joint name="${prefix}_joint_6">
-        <command_interface name="position"/>
-        <state_interface name="position"/>
-        <state_interface name="velocity"/>
-      </joint>
+    <ros2_control name="${name}" type="fake_components/GenericSystem">
     </ros2_control>
   </xacro:macro>

File: niryo_one_description/urdf/niryo_one_gripper.urdf.xacro (robot description, xacro)
@@ -89,5 +89,4 @@
                effort="1"
                velocity="5"/>
-        <mimic joint="${prefix}_gripper_joint" multiplier="1" offset="0" />
     </joint>
     <!-- Mors 2 -->
@@ -136,14 +135,5 @@
         <mimic joint="${prefix}_joint_base_to_mors_1" multiplier="1" offset="0" />
     </joint>
-    <ros2_control name="${prefix}_gripper" type="actuator">
-      <hardware>
-        <plugin>niryo_one_driver/NiryoOneActuatorInterface</plugin>
-      </hardware>
-      <joint name="${prefix}_joint_base_to_mors_1">
-        <command_interface name="position"/>
-        <state_interface name="position"/>
-        <state_interface name="velocity"/>
-        <state_interface name="effort"/>
-      </joint>
+    <ros2_control name="${prefix}_gripper" type="test_actuator">
     </ros2_control>
     <xacro:macro name="SimpleTransmissionEffort" params="joint n">
