Commit message: Remove unnecessary stuff

File: niryo_one_moveit_config/srdf/niryo_two.srdf.xacro (robot description, xacro)
@@ -36,26 +36,4 @@
         <group name="b_bot"/>
     </group>
-    <group name="a_bot_tool">
-        <link name="a_bot_base_gripper_1"/>
-        <joint name="a_bot_joint_to_gripper"/>
-        <joint name="a_bot_joint_base_to_mors_1"/>
-    </group>
-    <group_state name="close" group="a_bot_tool">
-        <joint name="a_bot_joint_base_to_mors_1" value="-0.01"/>
-    </group_state>
-    <group_state name="open" group="a_bot_tool">
-        <joint name="a_bot_joint_base_to_mors_1" value="0.007"/>
-    </group_state>
-    <group name="b_bot_tool">
-        <link name="b_bot_base_gripper_1"/>
-        <joint name="b_bot_joint_to_gripper"/>
-        <joint name="b_bot_joint_base_to_mors_1"/>
-    </group>
-    <group_state name="close" group="b_bot_tool">
-        <joint name="b_bot_joint_base_to_mors_1" value="-0.01"/>
-    </group_state>
-    <group_state name="open" group="b_bot_tool">
-        <joint name="b_bot_joint_base_to_mors_1" value="0.007"/>
-    </group_state>
     <!--VIRTUAL JOINT Purpose this element defines a virtual joint between a robot link and an external frame of reference (considered fixed with respect to the robot)-->
     <virtual_joint name="a_bot_joint_world" type="fixed" parent_frame="world" child_link="a_bot_base_link"/>

Commit message: Pick and Place initial commit

File: niryo_one_moveit_config/srdf/niryo_two.srdf.xacro (robot description, xacro)
@@ -36,4 +36,18 @@
         <group name="b_bot"/>
     </group>
+    <group_state name="resting" group="niryo_two">
+        <joint name="a_bot_joint_1" value="0" />
+        <joint name="a_bot_joint_2" value="0.64" />
+        <joint name="a_bot_joint_3" value="-1.38" />
+        <joint name="a_bot_joint_4" value="0" />
+        <joint name="a_bot_joint_5" value="0" />
+        <joint name="a_bot_joint_6" value="0" />
+        <joint name="b_bot_joint_1" value="0" />
+        <joint name="b_bot_joint_2" value="0.64" />
+        <joint name="b_bot_joint_3" value="-1.38" />
+        <joint name="b_bot_joint_4" value="0" />
+        <joint name="b_bot_joint_5" value="0" />
+        <joint name="b_bot_joint_6" value="0" />
+    </group_state>
     <!--VIRTUAL JOINT Purpose this element defines a virtual joint between a robot link and an external frame of reference (considered fixed with respect to the robot)-->
     <virtual_joint name="a_bot_joint_world" type="fixed" parent_frame="world" child_link="a_bot_base_link"/>
